File: src/Nano2UNO-Adapter-5V.kicad_sch (KiCad schematic)
At the start: 10 parts, among them J1 ESW-108-33-L-S, J2 ESW-110-33-L-S, J3 ESW-108-33-L-S, J4 ESW-106-33-L-S, J5 PPPC151LFBN-RC, J6 PPPC151LFBN-RC, J7 TSW-103-15-L-D, J8 PJ-102A, SW1 1825910-6

Commit message: Changed RST to RESET and REF to AREF. Tweaked README and production file creation instructions.
Changed lines of the file:
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@@
   (title_block
     (title "Nano2UNO Adapter 5V")
-    (date "2023-12-30")
+    (date "2023-12-31")
     (rev "0.0.1")
     (company "Designer: C. M. Bulliner")
